File: Shield/Shield.kicad_pcb (KiCad board)
At the start: 2 copper layers, 68.6 x 53.3 mm, 22 parts, among them P1 Power, P2 Analog, P3 Digital, P4 Digital, P5 CONN_01X01, P6 CONN_01X01, P7 CONN_01X01, P8 CONN_01X01

Commit message: ARDUINO V2
Parts:
- moved B1 1.41 mm to (135.0, 83.4)
Routing:
- net GND: track 40.3 -> 0.69 mm
- net +5V: track 169.9 -> 188.8 mm
- net ADC: track 25.6 -> 21.4 mm
- net IN-: track 31.7 -> 34.3 mm
- net Rx: track 17.8 -> 19.5 mm
- net Tx: track 17.8 -> 19.0 mm
- net DATA: track 13.2 -> 12.2 mm
- net CLK: track 13.2 -> 12.2 mm
- net SWITCH: track 13.2 -> 12.2 mm
